File: anderson_distribution_board.kicad_pcb (KiCad board)
At the start: 2 copper layers, 65 x 20 mm, 5 parts, among them J1 Anderson_two_redblack, J2 Anderson_two_redblack, J3 Anderson_two_redblack, J4 Anderson_two_redblack, J5 Anderson_two_redblack

Commit message: Polish and add gerbers
Other:
- board text added: "v1.0"
Changed lines of the file:
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@@
     (area 0 0 0 0)
     (thickness 1.6)
-    (drawings 4)
+    (drawings 5)
     (tracks 0)
     (zones 0)
@@
   (page A4)
   (layers
-    (0 F.Cu signal)
-    (31 B.Cu signal)
+    (0 F.Cu signal hide)
+    (31 B.Cu signal hide)
     (32 B.Adhes user)
     (33 F.Adhes user)
@@
       (net 2 "Net-(J1-Pad2)"))
   )
+  (gr_text v1.0 (at 101.5 77 90) (layer B.SilkS)
+    (effects (font (size 4 4) (thickness 0.7)) (justify mirror))
+  )
   (gr_line (start 90 67) (end 155 67) (layer Edge.Cuts) (width 0.15))
